File: Brooder.kicad_pcb (KiCad board)
At the start: 2 copper layers, 54 parts, among them J1 Heater, J11 Speaker OUT, J12 Encoder IN, J13 Serial Debug, J14 3.3V IN, J15 12V IN, J2 Electronics Fan, J3 Chamber Fan, J4 Lights, J5 Ambient SNSR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

Commit message: Added diode to chamber fan
Parts:
- added D2: 1N5819WS, Diode_SMD:D_SOD-323, F.Cu at (42.2, 72.5)
- U5: footprint Package_TO_SOT_THT:TO-92_Inline -> Sensor:DS18B20_SMD
Routing:
- net +12V: track 188.8 -> 196.6 mm
- net GND: track 0.00 -> 6.55 mm
