File: Brooder.kicad_sch (KiCad schematic)
At the start: 54 parts, among them J1 Heater, J11 Speaker OUT, J12 Encoder IN, J13 Serial Debug, J14 3.3V IN, J15 12V IN, J2 Electronics Fan, J3 Chamber Fan, J4 Lights, J5 Ambient SNSR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

Commit message: Added diode to chamber fan
Parts:
- added D2: 1N5819WS, Diode_SMD:D_SOD-323, symbol Diode:1N5819WS
- U5: footprint Package_TO_SOT_THT:TO-92_Inline -> Sensor:DS18B20_SMD
Connections:
- net +12V: now also D2.1 (K)
- net GND: now also D2.2 (A)
Changed lines of the file:
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@@
 	)
 	(junction
+		(at 242.57 50.8)
+		(diameter 0)
+		(color 0 0 0 0)
+	)
+	(junction
 		(at 257.81 116.84)
 		(diameter 0)
@@
 	)
 	(junction
+		(at 242.57 43.18)
+		(diameter 0)
+		(color 0 0 0 0)
+	)
+	(junction
 		(at 62.23 177.8)
 		(diameter 0)
@@
 	(wire
 		(pts
+			(xy 242.57 43.18) (xy 238.76 43.18)
+		)
+		(stroke
+			(width 0)
+			(type default)
+		)
+	)
+	(wire
+		(pts
 			(xy 222.25 95.25) (xy 210.82 95.25)
 		)
@@
 	(wire
 		(pts
-			(xy 252.73 50.8) (xy 240.03 50.8)
+			(xy 252.73 50.8) (xy 242.57 50.8)
 		)
 		(stroke
@@
 	(wire
 		(pts
-			(xy 252.73 43.18) (xy 238.76 43.18)
+			(xy 252.73 43.18) (xy 242.57 43.18)
 		)
 		(stroke
@@
 	(wire
 		(pts
+			(xy 242.57 50.8) (xy 240.03 50.8)
+		)
+		(stroke
+			(width 0)
+			(type default)
+		)
+	)
+	(wire
+		(pts
 			(xy 204.47 101.6) (xy 212.09 101.6)
 		)
@@
 			)
 		)
-		(property "Footprint" "Package_TO_SOT_THT:TO-92_Inline"
+		(property "Footprint" "Sensor:DS18B20_SMD"
 			(at 121.92 58.42 0)
 			(effects
@@
 					(unit 1)
 				)
+			)
+		)
+	)
+	(symbol
+		(lib_id "Diode:1N5819WS")
+		(at 242.57 46.99 90)
+		(unit 1)
+		(exclude_from_sim no)
+		(in_bom yes)
+		(on_board yes)
+		(dnp no)
+		(fields_autoplaced yes)
+		(property "Reference" "D2"
+			(at 245.11 46.0374 90)
+			(effects
+				(font
+					(size 1.27 1.27)
+				)
+				(justify right)
+			)
+		)
+		(property "Value" "1N5819WS"
+			(at 245.11 48.5774 90)
+			(effects
+				(font
+					(size 1.27 1.27)
+				)
+				(justify right)
+			)
+		)
+		(property "Footprint" "Diode_SMD:D_SOD-323"
+			(at 247.015 46.99 0)
+			(effects
+				(font
+					(size 1.27 1.27)
+				)
+				(hide yes)
+			)
+		)
+		(property "Datasheet" "https://datasheet.lcsc.com/lcsc/2204281430_Guangdong-Hottech-1N5819WS_C191023.pdf"
+			(at 242.57 46.99 0)
+			(effects
+				(font
+					(size 1.27 1.27)
+				)
+				(hide yes)
+			)
+		)
+		(property "Description" "40V 600mV@1A 1A SOD-323 Schottky Barrier Diodes, SOD-323"
+			(at 242.57 46.99 0)
+			(effects
+				(font
+					(size 1.27 1.27)
+				)
+				(hide yes)
+			)
+		)
+		(pin "1"
+		)
+		(pin "2"
+		)
+		(instances
+			(project "Brooder"
+				(path "/9041d520-f59c-4387-8e49-bb57372058b5"
+					(reference "D2")
+					(unit 1)
+				)
